File: System Connector Board/SysCon.kicad_pcb (KiCad board)
At the start: 2 copper layers, 100 x 60 mm, 11 parts, among them U1 GAL16V8

Commit message: Add files via upload
Routing:
- net /SNES.PA1: track 46.5 -> 44.7 mm, vias 2 -> 0
- net /SNES.D7: track 46.8 -> 45.2 mm
- net /SNES.~{PAWR}: track 45.7 -> 44.7 mm, vias 2 -> 0
- net /SNES.Refresh: track 45.8 -> 44.7 mm, vias 2 -> 0
- net /SNES.~{PARD}: track 45.7 -> 44.7 mm
- net /SNES.BA5.Mod: track 22.3 -> 21.4 mm
- net /SNES.BA5: track 29.0 -> 29.9 mm
- net /SNES.Expand: track 45.4 -> 44.7 mm
- net /SNES.BA3: track 50.8 -> 50.2 mm
- net /SNES.R_Audio: track 45.4 -> 44.9 mm, vias 2 -> 0
- net /SNES.A4: track 51.3 -> 50.7 mm
